Commit message: fixed kmr iiwa description

File: urdf/kmr.xacro (robot description, xacro)
@@ -2,47 +2,15 @@
 <robot xmlns:xacro="http://www.ros.org/wiki/xacro">
   <xacro:macro name="kmr" params="robot_name">
-    <link name="odom" />
-    <joint name="odom_x_joint" type="prismatic">
-      <parent link="odom"/>
-      <child link="odom_x_frame"/>
-      <axis xyz="1 0 0"/>
-     <!-- limits chosen heuristically
-          lower/upper: +-1km to create a quasi limitless prismatic joint
-          velocity: slow walking speed is 3-4km/hour ~= 1m/s
-          effort: reach max speed within 1s, Boxy has a mass of 200kg, so Fmax=200kg*1m/s2 -->
-      <limit lower="-1000" upper="1000" velocity="1" effort="200"/>
-    </joint>
-    <link name="odom_x_frame" />
-    <joint name="odom_y_joint" type="prismatic">
-      <parent link="odom_x_frame"/>
-      <child link="odom_y_frame"/>
-      <axis xyz="0 1 0"/>
-      <!-- limits chosen heuristically
-           lower/upper: +-1km to create a quasi limitless prismatic joint
-           velocity: slow walking speed is 3-4km/hour ~= 1m/s
-           effort: reach max speed within 1s, Boxy has a mass of 200kg, so Fmax=200kg*1m/s2 -->
-      <limit lower="-1000" upper="1000" velocity="1" effort="200"/>
-    </joint>
-    <link name="odom_y_frame" />
-    <joint name="odom_z_joint" type="continuous">
-      <parent link="odom_y_frame"/>
-      <child link="base_footprint"/>
-      <axis xyz="0 0 1"/>
-      <!-- limits chosen heuristically
-           velocity: one slow complete turn around in 5-6s, so 6.2rad/6s ~= 1rad/s
-           effort: reach max speed within 1s, Boxy has a mass of 200kg and a diagonale of 1m, so Fmax=200kg*1m*1m/s2 -->
-      <limit velocity="1" effort="200"/>
-    </joint>
-    <link name="base_footprint"/>
+  <!--   <link name="base_footprint"/>
     <joint name="base_joint" type="fixed">
       <parent link="base_footprint"/>
       <child link="base_link"/>
       <origin xyz="0 0 0" rpy="0 0 0"/>
-    </joint>
+    </joint> -->
     <link name="base_link">
       <visual>
         <origin xyz="0 0 0" rpy="0 0 ${pi}"/>
         <geometry>
-          <mesh filename="package://kmr_iiwa_description/meshes/kmp200_3ds_export.dae"/>
+          <mesh filename="package://iai_kmr_iiwa_description/meshes/kmp200_3ds_export.dae"/>
         </geometry>
         <material name="Grey"/>
@@ -51,9 +19,21 @@
         <origin xyz="0 0 0" rpy="0 0 ${pi}"/>
         <geometry>
-          <mesh filename="package://kmr_iiwa_description/meshes/kmp200_export.stl"/>
+          <mesh filename="package://iai_kmr_iiwa_description/meshes/kmp200_export.stl"/>
         </geometry>
         <material name="Grey"/>
       </collision>
     </link>
+  <!--   <joint name="back_laser_joint" type="fixed">
+      <parent link="base_footprint"/>
+      <child link="back_laser"/>
+      <origin xyz="-0.464, 0.256, 0.140" rpy="0.000, -0.000, 2.356"/>
+    </joint>
+    <link name="back_laser"/>
+    <joint name="front_laser_joint" type="fixed">
+      <parent link="base_footprint"/>
+      <child link="front_laser"/>
+      <origin xyz="0.464, -0.256, 0.140" rpy="0.000, 0.000, -0.785"/>
+    </joint>
+    <link name="front_laser"/> -->
   </xacro:macro>
 </robot>

File: urdf/kmr_iiwa_with_odom_joints.urdf.xacro (robot description, xacro)
@@ -4,5 +4,5 @@
   <!-- <xacro:include filename="$(find kmr_iiwa_description)/urdf/materials.xacro" /> -->
   <!--Import the lbr iiwa macro -->
-  <xacro:include filename="$(find iai_kmr_iiwa_description)/urdf/kmr_iiwa.xacro"/>
+  <xacro:include filename="$(find iai_kmr_iiwa_description)/urdf/kmr_iiwa_with_odom_joints.xacro"/>
   <xacro:arg name="hardware_interface" default="PositionJointInterface"/>
   <xacro:arg name="robot_name" default="kmr_iiwa"/>

File: urdf/kmr_iiwa_with_odom_joints.xacro (robot description, xacro)
@@ -12,5 +12,5 @@
   <!--Import the lbr iiwa macro -->
   <xacro:include filename="$(find iiwa_description)/urdf/iiwa14.xacro"/>
-  <xacro:include filename="$(find iai_kmr_iiwa_description)/urdf/kmr.xacro"/>
+  <xacro:include filename="$(find iai_kmr_iiwa_description)/urdf/kmr_with_odom_joints.xacro"/>
   <xacro:arg name="hardware_interface" default="PositionJointInterface"/>
   <xacro:arg name="robot_name" default="kmr_iiwa"/>
