Commit message: Fix description and launch files

File: iai_kmr_iiwa_description/urdf/kmr_iiwa.urdf.xacro (robot description, xacro)
@@ -4,7 +4,7 @@
   <!-- <xacro:include filename="$(find kmr_iiwa_description)/urdf/materials.xacro" /> -->
   <!--Import the lbr iiwa macro -->
-  <xacro:include filename="$(find iai_kmr_iiwa_description)/urdf/kmr_iiwa.xacro"/>
-  <xacro:arg name="hardware_interface" default="PositionJointInterface"/>
-  <xacro:arg name="robot_name" default="kmr_iiwa"/>
+  <xacro:include filename="$(find iai_kmr_iiwa_description)/urdf/kmr_iiwa.xacro" />
+  <xacro:arg name="hardware_interface" default="PositionJointInterface" />
+  <xacro:arg name="robot_name" default="kmr_iiwa" />
   <!--iiwa-->
   <xacro:kmr_iiwa hardware_interface="$(arg hardware_interface)" robot_name="$(arg robot_name)">

File: iai_kmr_iiwa_description/urdf/kmr_iiwa.xacro (robot description, xacro)
@@ -1,6 +1,4 @@
 <?xml version="1.0"?>
 <robot xmlns:xacro="http://www.ros.org/wiki/xacro">
-  <xacro:include filename="$(find iiwa_description)/urdf/iiwa14.xacro" />
-  <!-- <xacro:include filename="$(find ur_description)/urdf/ur5.urdf.xacro" /> -->
   <xacro:include filename="$(find iai_kms_40_description)/urdf/kms_40.urdf.xacro"/>
   <xacro:include filename="$(find iai_adapters_description)/urdf/adapter_fwa050_wsg50.urdf.xacro"/>
@@ -75,19 +73,19 @@
       <origin xyz="0 0 0" rpy="0 0 ${pi}" />
     </joint>
-    <kms_40_xacro parent="kms_mounting_plate" prefix="">
+    <xacro:kms_40_xacro parent="kms_mounting_plate" prefix="">
       <origin xyz="0 0 0" rpy="0 0 ${pi}" />
-    </kms_40_xacro>
-    <adapter_kms40_fwk050_xacro parent="kms40_frame_out" prefix="">
+    </xacro:kms_40_xacro>
+    <xacro:adapter_kms40_fwk050_xacro parent="kms40_frame_out" prefix="">
       <origin xyz="0 0 0" rpy="0 0 0" />
-    </adapter_kms40_fwk050_xacro>
-    <fwk_fwa_050_xacro parent="adapter_kms40_fwk050_frame_out" prefix="">
+    </xacro:adapter_kms40_fwk050_xacro>
+    <xacro:fwk_fwa_050_xacro parent="adapter_kms40_fwk050_frame_out" prefix="">
       <origin xyz="0 0 0" rpy="0 0 0" />
-    </fwk_fwa_050_xacro>
-    <adapter_fwa050_wsg50_xacro parent="fwk_fwa_050_frame_out" prefix="">
+    </xacro:fwk_fwa_050_xacro>
+    <xacro:adapter_fwa050_wsg50_xacro parent="fwk_fwa_050_frame_out" prefix="">
       <origin xyz="0 0 0.0" rpy="0 0 0" />
-    </adapter_fwa050_wsg50_xacro>
-    <wsg_50_xacro name="gripper" parent="adapter_fwa050_wsg50_frame_out">
+    </xacro:adapter_fwa050_wsg50_xacro>
+    <xacro:wsg_50_xacro name="gripper" parent="adapter_fwa050_wsg50_frame_out">
       <origin xyz="0 0 0" rpy="0 0 3.14159265359"/>
-    </wsg_50_xacro>
+    </xacro:wsg_50_xacro>
     <link name="camera_holder_link">
       <visual>

File: iai_kmr_iiwa_description/urdf/kmr_iiwa_with_odom_joints.urdf.xacro (robot description, xacro)
@@ -4,9 +4,41 @@
   <!-- <xacro:include filename="$(find kmr_iiwa_description)/urdf/materials.xacro" /> -->
   <!--Import the lbr iiwa macro -->
-  <xacro:include filename="$(find iai_kmr_iiwa_description)/urdf/kmr_iiwa_with_odom_joints.xacro"/>
-  <xacro:arg name="hardware_interface" default="PositionJointInterface"/>
-  <xacro:arg name="robot_name" default="kmr_iiwa"/>
+  <xacro:include filename="$(find iai_kmr_iiwa_description)/urdf/kmr_iiwa.xacro" />
+  <xacro:arg name="hardware_interface" default="PositionJointInterface" />
+  <xacro:arg name="robot_name" default="kmr_iiwa" />
   <!--iiwa-->
   <xacro:kmr_iiwa hardware_interface="$(arg hardware_interface)" robot_name="$(arg robot_name)">
   </xacro:kmr_iiwa>
+  <link name="odom" />
+  <joint name="odom_x_joint" type="prismatic">
+    <parent link="odom" />
+    <child link="odom_x_frame" />
+    <axis xyz="1 0 0" />
+    <!-- limits chosen heuristically
+        lower/upper: +-1km to create a quasi limitless prismatic joint
+        velocity: slow walking speed is 3-4km/hour ~= 1m/s
+        effort: reach max speed within 1s, Boxy has a mass of 200kg, so Fmax=200kg*1m/s2 -->
+    <limit lower="-1000" upper="1000" velocity="1" effort="200" />
+  </joint>
+  <link name="odom_x_frame" />
+  <joint name="odom_y_joint" type="prismatic">
+    <parent link="odom_x_frame" />
+    <child link="odom_y_frame" />
+    <axis xyz="0 1 0" />
+    <!-- limits chosen heuristically
+          lower/upper: +-1km to create a quasi limitless prismatic joint
+          velocity: slow walking speed is 3-4km/hour ~= 1m/s
+          effort: reach max speed within 1s, Boxy has a mass of 200kg, so Fmax=200kg*1m/s2 -->
+    <limit lower="-1000" upper="1000" velocity="1" effort="200" />
+  </joint>
+  <link name="odom_y_frame" />
+  <joint name="odom_z_joint" type="continuous">
+    <parent link="odom_y_frame" />
+    <child link="base_link" />
+    <axis xyz="0 0 1" />
+    <!-- limits chosen heuristically
+          velocity: one slow complete turn around in 5-6s, so 6.2rad/6s ~= 1rad/s
+          effort: reach max speed within 1s, Boxy has a mass of 200kg and a diagonale of 1m, so Fmax=200kg*1m*1m/s2 -->
+    <limit velocity="1" effort="200" />
+  </joint>
 </robot>
