Commit message: fixed kmr iiwa launch files

File: iai_kmr_iiwa_description/urdf/kmr_iiwa.xacro (robot description, xacro)
@@ -73,5 +73,5 @@
       <parent link="iiwa_link_ee" />
       <child link="kms_mounting_plate" />
-      <origin xyz="0 0 0" rpy="0 0 ${pi}" />
+      <origin xyz="0 0 0" rpy="0 0 0" />
     </joint>
     <kms_40_xacro parent="kms_mounting_plate" prefix="">

Commit message: calibrated camera poses

File: iai_kmr_iiwa_description/urdf/kmr_iiwa.xacro (robot description, xacro)
@@ -108,6 +108,6 @@
     </joint>
     <link name="camera_link"/>
-    <joint name="gripper_to_camera_joint" type="fixed">
-      <parent link="gripper_base_link" />
+    <joint name="iiwa_link_ee_to_camera_joint" type="fixed">
+      <parent link="iiwa_link_ee" />
       <child link="camera_link" />
       <!--Calib_errors = [0.003425, 0.2069, 0.00611, 0.42678]
@@ -116,5 +116,5 @@
       <!-- from ur5_base_link origin xyz="0.002956 -0.066498 0.060947" rpy="0.204429 6.281375 3.127197"/-->
       <!-- calib errors: 0.00311, 0.24373, 0.00688, 0.4558 -->
-      <origin xyz="0.002956 -0.066498 0.060947" rpy="0.204429 6.281375 3.127197" />
+      <origin xyz="0.001329 -0.066190 0.111783" rpy="0.231224 6.279694 3.148548"/>
     </joint>
     <link name="rs_camera_link"/>
@@ -122,5 +122,6 @@
       <parent link="camera_link" />
       <child link="rs_camera_link" />
-      <origin xyz="-0.017993 -0.107556 0.017699" rpy="6.270618 4.930698 1.578454"/>
+      <!-- <origin xyz="-0.017993 -0.107556 0.017699" rpy="6.270618 4.930698 1.578454"/> -->
+      <origin xyz="-0.018594 -0.105693 0.017161" rpy="6.271141 4.940698 1.579879"/>
     </joint>
     <joint name="wrist_collision_joint" type="fixed">

Commit message: rotated kmrs camera by 180 degree

File: iai_kmr_iiwa_description/urdf/kmr_iiwa.xacro (robot description, xacro)
@@ -87,5 +87,5 @@
     </xacro:adapter_fwa050_wsg50_xacro> -->
     <xacro:wsg_50_xacro name="gripper" parent="fwk_fwa_050_frame_out">
-      <origin xyz="0 0 0" rpy="0 0 0"/>
+      <origin xyz="0 0 0" rpy="0 0 ${pi}"/>
     </xacro:wsg_50_xacro>
     <link name="camera_holder_link">
@@ -117,5 +117,8 @@
       <!-- from ur5_base_link origin xyz="0.002956 -0.066498 0.060947" rpy="0.204429 6.281375 3.127197"/-->
       <!-- calib errors: 0.00311, 0.24373, 0.00688, 0.4558 -->
-      <origin xyz="0.001329 -0.066190 0.111783" rpy="0.231224 6.279694 3.148548"/>
+      <!-- what we calibrated with alexis, relative to ee link -->
+      <!-- <origin xyz="0.001329 -0.066190 0.111783" rpy="0.231224 6.279694 3.148548"/>  -->
+      <!-- from tf lookup shifted to gripper_base_link -->
+      <origin xyz="-0.00132899999999 0.06619 0.071683" rpy="0.231224 -0.00349130717959 0.00695534641"/>
     </joint>
     <link name="rs_camera_link"/>
