Commit message: fixed kmr base rotation

File: iai_kmr_iiwa_description/urdf/kmr.xacro (robot description, xacro)
@@ -10,5 +10,5 @@
     <link name="base_link">
       <visual>
-        <origin xyz="0 0 0" rpy="0 0 ${pi}"/>
+        <origin xyz="0 0 0" rpy="0 0 0"/>
         <geometry>
           <mesh filename="package://iai_kmr_iiwa_description/meshes/kmp200_3ds_export.dae"/>
@@ -17,5 +17,5 @@
       </visual>
       <collision>
-        <origin xyz="0 0 0" rpy="0 0 ${pi}"/>
+        <origin xyz="0 0 0" rpy="0 0 0"/>
         <geometry>
           <mesh filename="package://iai_kmr_iiwa_description/meshes/kmp200_export.stl"/>
@@ -24,16 +24,16 @@
       </collision>
     </link>
-  <!--   <joint name="back_laser_joint" type="fixed">
-      <parent link="base_footprint"/>
+    <joint name="back_laser_joint" type="fixed">
+      <parent link="base_link"/>
       <child link="back_laser"/>
-      <origin xyz="-0.464, 0.256, 0.140" rpy="0.000, -0.000, 2.356"/>
+      <origin xyz="-0.464 0.256 0.140" rpy="0.000 -0.000 2.356"/>
     </joint>
     <link name="back_laser"/>
     <joint name="front_laser_joint" type="fixed">
-      <parent link="base_footprint"/>
+      <parent link="base_link"/>
       <child link="front_laser"/>
-      <origin xyz="0.464, -0.256, 0.140" rpy="0.000, 0.000, -0.785"/>
+      <origin xyz="0.464 -0.256 0.140" rpy="0.000 0.000 -0.785"/>
     </joint>
-    <link name="front_laser"/> -->
+    <link name="front_laser"/>
   </xacro:macro>
 </robot>

File: iai_kmr_iiwa_description/urdf/kmr_iiwa.xacro (robot description, xacro)
@@ -26,5 +26,5 @@
       <parent link="base_link" />
       <child link="angle_adapter_base" />
-      <origin xyz="-0.363 0 0.7" rpy="0 0 ${-pi/2}" />
+      <origin xyz="0.363 0 0.7" rpy="0 0 ${pi/2}" />
     </joint>
     <link name="angle_adapter_base">

Commit message: [description] low-res mesh for base collision

File: iai_kmr_iiwa_description/urdf/kmr.xacro (robot description, xacro)
@@ -19,5 +19,5 @@
         <origin xyz="0 0 0" rpy="0 0 0"/>
         <geometry>
-          <mesh filename="package://iai_kmr_iiwa_description/meshes/kmp200_export.stl"/>
+          <mesh filename="package://iai_kmr_iiwa_description/meshes/kmp200_3ds_export_s.stl"/>
         </geometry>
         <material name="Grey"/>
