Commit message: added low res meshes and the correct one for link 7

File: iai_iiwa_description/urdf/iiwa14.xacro (robot description, xacro)
@@ -280,5 +280,5 @@
         <origin xyz="0 0 0" rpy="0 0 0"/>
         <geometry>
-          <mesh filename="package://iai_iiwa_description/meshes/iiwa14/visual/link_7.stl"/>
+          <mesh filename="package://iai_iiwa_description/meshes/iiwa14/visual/link_7-MF-Touch-pneumatisch.stl"/>
         </geometry>
         <material name="Grey"/>
@@ -287,5 +287,5 @@
         <origin xyz="0 0 0" rpy="0 0 0"/>
         <geometry>
-          <mesh filename="package://iai_iiwa_description/meshes/iiwa14/collision/link_7.stl"/>
+          <mesh filename="package://iai_iiwa_description/meshes/iiwa14/collision/link_7-MF-Touch-pneumatisch.stl"/>
         </geometry>
         <material name="Grey"/>

File: iai_kmr_iiwa_description/urdf/kmr_iiwa.xacro (robot description, xacro)
@@ -60,5 +60,5 @@
       <origin xyz="0 0 0.00" rpy="0 0 ${-pi/2}" />
     </xacro:iiwa14>
-    <link name="kms_mounting_plate">
+ <!--    <link name="kms_mounting_plate">
       <visual>
         <geometry>
@@ -75,16 +75,17 @@
     <xacro:kms_40_xacro parent="kms_mounting_plate" prefix="">
       <origin xyz="0 0 0" rpy="0 0 ${pi}" />
-    </xacro:kms_40_xacro>
+    </xacro:kms_40_xacro> -->
+<!--
     <xacro:adapter_kms40_fwk050_xacro parent="kms40_frame_out" prefix="">
       <origin xyz="0 0 0" rpy="0 0 0" />
-    </xacro:adapter_kms40_fwk050_xacro>
-    <xacro:fwk_fwa_050_xacro parent="adapter_kms40_fwk050_frame_out" prefix="">
-      <origin xyz="0 0 0" rpy="0 0 0" />
+    </xacro:adapter_kms40_fwk050_xacro> -->
+    <xacro:fwk_fwa_050_xacro parent="iiwa_link_ee" prefix="">
+      <origin xyz="0 0 0.026" rpy="0 0 0" />
     </xacro:fwk_fwa_050_xacro>
-    <xacro:adapter_fwa050_wsg50_xacro parent="fwk_fwa_050_frame_out" prefix="">
+<!--     <xacro:adapter_fwa050_wsg50_xacro parent="fwk_fwa_050_frame_out" prefix="">
       <origin xyz="0 0 0.0" rpy="0 0 0" />
-    </xacro:adapter_fwa050_wsg50_xacro>
-    <xacro:wsg_50_xacro name="gripper" parent="adapter_fwa050_wsg50_frame_out">
-      <origin xyz="0 0 0" rpy="0 0 3.14159265359"/>
+    </xacro:adapter_fwa050_wsg50_xacro> -->
+    <xacro:wsg_50_xacro name="gripper" parent="fwk_fwa_050_frame_out">
+      <origin xyz="0 0 0" rpy="0 0 0"/>
     </xacro:wsg_50_xacro>
     <link name="camera_holder_link">
@@ -125,5 +126,5 @@
     </joint>
     <joint name="wrist_collision_joint" type="fixed">
-      <parent link="adapter_kms40_fwk050_frame_in" />
+      <parent link="iiwa_link_ee" />
       <child link="wrist_collision" />
       <origin xyz="0 0 -0.005" rpy="0 0 0" />
